Commit message: Add explorer_state

File: candybot5_description/urdf/turtlebot3_burger.urdf.xacro (robot description, xacro)
@@ -115,5 +115,5 @@
   <joint name="sonar_front_joint1" type="fixed">
     <axis xyz="0 1 0" />
-    <origin rpy="0 0 0" xyz="0.05 0.04 0.03" />
+    <origin rpy="0 0 0" xyz="-0.11 0.04 0.03" />
     <parent link="base_footprint"/>
     <child link="base_sonar_front1"/>
@@ -140,5 +140,5 @@
   <joint name="sonar_front_joint2" type="fixed">
     <axis xyz="0 1 0" />
-    <origin rpy="0 0 0" xyz="0.05 -0.04 0.03" />
+    <origin rpy="0 0 0" xyz="-0.11 -0.04 0.03" />
     <parent link="base_footprint"/>
     <child link="base_sonar_front2"/>
@@ -165,5 +165,5 @@
   <joint name="infrared_front_joint1" type="fixed">
     <axis xyz="0 1 0" />
-    <origin rpy="0 1.57 0" xyz="0.09 0.09 0.02" />
+    <origin rpy="0 1.57 0" xyz="-0.15 0.09 0.02" />
     <parent link="base_footprint"/>
     <child link="base_infrared_front1"/>
@@ -190,5 +190,5 @@
   <joint name="infrared_front_joint2" type="fixed">
     <axis xyz="0 1 0" />
-    <origin rpy="0 1.57 0" xyz="0.09 -0.09 0.02" />
+    <origin rpy="0 1.57 0" xyz="-0.15 -0.09 0.02" />
     <parent link="base_footprint"/>
     <child link="base_infrared_front2"/>
